File: micro-sd-spi-breakout-module.kicad_sch (KiCad schematic)
At the start: 2 parts, among them J1 Micro_SD_Card_Det1, J2 Conn_01x06_Pin

Commit message: Schematic, Routing and Silkscreen Completed
Parts:
- removed J1: Micro_SD_Card_Det1, symbol Connector:Micro_SD_Card_Det1
- removed J2: Conn_01x06_Pin, symbol Connector:Conn_01x06_Pin
- added C1: 10uF, symbol Device:C
- added C2: 100nF, symbol Device:C
- added J1: Conn_01x07_Pin, symbol Connector:Conn_01x07_Pin
- added R1, R2: 10K, symbol Device:R
- added U1: TF-SMD_TF-PUSH, symbol TF-SMD_TF-PUSH_TF_PUSH_C393941:TF-SMD_TF-PUSH
Connections:
- net CD_DET: now also J1.6 (Pin_6), R1.2, U1.9
- net CS: now also J1.2 (Pin_2), U1.2
- net GND: now also C1.2, C2.2, J1.7 (Pin_7), U1.10, U1.11, U1.12, U1.13, U1.6
- net MISO: now also J1.5 (Pin_5), R2.2, U1.7
- net MOSI: now also J1.3 (Pin_3), U1.3
- net SCK: now also J1.4 (Pin_4), U1.5
- net SD_3V3: now also C1.1, C2.1, J1.1 (Pin_1), R1.1, R2.1, U1.4

Commit message: Schematic, Routing and Silkscreen Completed
Parts:
- C1: footprint (none) -> 10uF-Cap:C0603_CL10A106KP8NNNC_C19702
- C2: footprint (none) -> 100nF-Cap:C0603_CC0603JRX7R9BB104_C91183
- J1: footprint (none) -> Connector_PinHeader_2.54mm:PinHeader_1x07_P2.54mm_Horizontal
- R1, R2: footprint (none) -> 10K-Res:R0603_FRC0603F1001TS_C2907002
- U1: footprint (none) -> Sd-Card-Holder:TF-SMD_TF-PUSH_TF_PUSH_C393941
Connections:
- net CD_DET: now also J1.2 (Pin_2); no longer J1.6 (Pin_6)
- net CS: now also J1.6 (Pin_6); no longer J1.2 (Pin_2)
- net GND: now also J1.1 (Pin_1); no longer J1.7 (Pin_7)
- net MISO: now also J1.3 (Pin_3); no longer J1.5 (Pin_5)
- net MOSI: now also J1.5 (Pin_5); no longer J1.3 (Pin_3)
- net SD_3V3: now also J1.7 (Pin_7); no longer J1.1 (Pin_1)
Changed lines of the file:
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@@
 			)
 		)
-		(property "Footprint" ""
+		(property "Footprint" "100nF-Cap:C0603_CC0603JRX7R9BB104_C91183"
 			(at 145.7452 81.915 0)
 			(hide yes)
@@
 		(lib_id "Connector:Conn_01x07_Pin")
 		(at 91.44 103.505 0)
-		(unit 1)
-		(body_style 1)
-		(exclude_from_sim no)
-		(in_bom yes)
-		(on_board yes)
-		(in_pos_files yes)
-		(dnp no)
-		(fields_autoplaced yes)
+		(mirror x)
+		(unit 1)
+		(body_style 1)
+		(exclude_from_sim no)
+		(in_bom yes)
+		(on_board yes)
+		(in_pos_files yes)
+		(dnp no)
 		(property "Reference" "J1"
-			(at 92.075 91.44 0)
+			(at 92.075 115.57 0)
 			(show_name no)
 			(do_not_autoplace no)
@@
 		)
 		(property "Value" "Conn_01x07_Pin"
-			(at 92.075 93.98 0)
-			(show_name no)
-			(do_not_autoplace no)
-			(effects
-				(font
-					(size 1.27 1.27)
-				)
-			)
-		)
-		(property "Footprint" ""
+			(at 92.075 113.03 0)
+			(show_name no)
+			(do_not_autoplace no)
+			(effects
+				(font
+					(size 1.27 1.27)
+				)
+			)
+		)
+		(property "Footprint" "Connector_PinHeader_2.54mm:PinHeader_1x07_P2.54mm_Horizontal"
 			(at 91.44 103.505 0)
 			(hide yes)
@@
 			)
 		)
-		(property "Footprint" ""
+		(property "Footprint" "10K-Res:R0603_FRC0603F1001TS_C2907002"
 			(at 141.732 103.505 90)
 			(hide yes)
@@
 			)
 		)
-		(property "Footprint" ""
+		(property "Footprint" "Sd-Card-Holder:TF-SMD_TF-PUSH_TF_PUSH_C393941"
 			(at 90.805 27.305 0)
 			(hide yes)
@@
 			)
 		)
-		(property "Footprint" ""
+		(property "Footprint" "10uF-Cap:C0603_CL10A106KP8NNNC_C19702"
 			(at 134.9502 81.915 0)
 			(hide yes)
@@
 			)
 		)
-		(property "Footprint" ""
+		(property "Footprint" "10K-Res:R0603_FRC0603F1001TS_C2907002"
 			(at 148.717 103.505 90)
 			(hide yes)

Commit message: Images
Other:
- note added: "PIN HEADERS"
- note added: "SD CARD SLOT"
- company: (none) -> HTRONICS
- title: (none) -> Micro SD SPI Breakout Module
- moved on the sheet: J1
Changed lines of the file:
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@@
 	(generator_version "10.0")
 	(paper "A4")
+	(title_block
+		(title "Micro SD SPI Breakout Module")
+		(date "2026-08-03")
+		(rev "V1.0")
+		(company "HTRONICS")
+		(comment 1 "Designed By - Harsha")
+	)
+	(text "PIN HEADERS"
+		(exclude_from_sim no)
+		(at 53.975 72.39 0)
+		(effects
+			(font
+				(size 5.08 5.08)
+				(thickness 1.016)
+				(bold yes)
+			)
+		)
+	)
+	(text "SD CARD SLOT"
+		(exclude_from_sim no)
+		(at 208.28 71.12 0)
+		(effects
+			(font
+				(size 5.08 5.08)
+				(thickness 1.016)
+				(bold yes)
+			)
+		)
+	)
 	(junction
 		(at 154.305 71.12)
@@
 	)
 	(junction
-		(at 108.585 114.935)
+		(at 77.47 115.57)
 		(diameter 0)
 		(color 0 0 0 0)
@@
 	)
 	(junction
-		(at 108.585 92.075)
+		(at 77.47 92.71)
 		(diameter 0)
 		(color 0 0 0 0)
@@
 	(wire
 		(pts
-			(xy 108.585 92.075) (xy 108.585 95.885)
+			(xy 77.47 92.71) (xy 77.47 96.52)
 		)
 		(stroke
@@
 	(wire
 		(pts
-			(xy 96.52 98.425) (xy 108.585 98.425)
+			(xy 65.405 99.06) (xy 77.47 99.06)
 		)
 		(stroke
@@
 	(wire
 		(pts
-			(xy 108.585 114.935) (xy 108.585 116.84)
+			(xy 77.47 115.57) (xy 77.47 117.475)
 		)
 		(stroke
@@
 	(wire
 		(pts
-			(xy 96.52 103.505) (xy 108.585 103.505)
+			(xy 65.405 104.14) (xy 77.47 104.14)
 		)
 		(stroke
@@
 	(wire
 		(pts
-			(xy 96.52 106.045) (xy 108.585 106.045)
+			(xy 65.405 106.68) (xy 77.47 106.68)
 		)
 		(stroke
@@
 	(wire
 		(pts
-			(xy 96.52 100.965) (xy 108.585 100.965)
+			(xy 65.405 101.6) (xy 77.47 101.6)
 		)
 		(stroke
@@
 	(wire
 		(pts
-			(xy 108.585 88.9) (xy 108.585 92.075)
+			(xy 77.47 89.535) (xy 77.47 92.71)
 		)
 		(stroke
@@
 	(wire
 		(pts
-			(xy 96.52 111.125) (xy 108.585 111.125)
-		)
-		(stroke
-			(width 0)
-			(type default)
-		)
-	)
-	(wire
-		(pts
-			(xy 108.585 111.125) (xy 108.585 114.935)
-		)
-		(stroke
-			(width 0)
-			(type default)
-		)
-	)
-	(wire
-		(pts
-			(xy 96.52 108.585) (xy 108.585 108.585)
-		)
-		(stroke
-			(width 0)
-			(type default)
-		)
-	)
-	(wire
-		(pts
-			(xy 108.585 95.885) (xy 96.52 95.885)
+			(xy 65.405 111.76) (xy 77.47 111.76)
+		)
+		(stroke
+			(width 0)
+			(type default)
+		)
+	)
+	(wire
+		(pts
+			(xy 77.47 111.76) (xy 77.47 115.57)
+		)
+		(stroke
+			(width 0)
+			(type default)
+		)
+	)
+	(wire
+		(pts
+			(xy 65.405 109.22) (xy 77.47 109.22)
+		)
+		(stroke
+			(width 0)
+			(type default)
+		)
+	)
+	(wire
+		(pts
+			(xy 77.47 96.52) (xy 65.405 96.52)
 		)
 		(stroke
@@
 	)
 	(label "SCK"
-		(at 108.585 103.505 180)
+		(at 77.47 104.14 180)
 		(effects
 			(font
@@
 	)
 	(label "CS"
-		(at 108.585 98.425 180)
+		(at 77.47 99.06 180)
 		(effects
 			(font
@@
 	)
 	(label "MISO"
-		(at 108.585 106.045 180)
+		(at 77.47 106.68 180)
 		(effects
 			(font
@@
 	)
 	(label "CD_DET"
-		(at 108.585 108.585 180)
+		(at 77.47 109.22 180)
 		(effects
 			(font
@@
 	)
 	(label "MOSI"
-		(at 108.585 100.965 180)
+		(at 77.47 101.6 180)
 		(effects
 			(font
@@
 	(symbol
 		(lib_id "Connector:Conn_01x07_Pin")
-		(at 91.44 103.505 0)
+		(at 60.325 104.14 0)
 		(mirror x)
 		(unit 1)
@@
 		(dnp no)
 		(property "Reference" "J1"
-			(at 92.075 115.57 0)
+			(at 60.96 116.205 0)
 			(show_name no)
 			(do_not_autoplace no)
@@
 		)
 		(property "Value" "Conn_01x07_Pin"
-			(at 92.075 113.03 0)
+			(at 60.96 113.665 0)
 			(show_name no)
 			(do_not_autoplace no)
@@
 		)
 		(property "Footprint" "Connector_PinHeader_2.54mm:PinHeader_1x07_P2.54mm_Horizontal"
-			(at 91.44 103.505 0)
+			(at 60.325 104.14 0)
 			(hide yes)
 			(show_name no)
@@
 		)
 		(property "Datasheet" ""
-			(at 91.44 103.505 0)
+			(at 60.325 104.14 0)
 			(hide yes)
 			(show_name no)
@@
 		)
 		(property "Description" "Generic connector, single row, 01x07, script generated"
-			(at 91.44 103.505 0)
+			(at 60.325 104.14 0)
 			(hide yes)
 			(show_name no)
@@
 	(symbol
 		(lib_id "power:+3V3")
-		(at 108.585 88.9 0)
+		(at 77.47 89.535 0)
 		(unit 1)
 		(body_style 1)
@@
 		(fields_autoplaced yes)
 		(property "Reference" "#PWR06"
-			(at 108.585 92.71 0)
+			(at 77.47 93.345 0)
 			(hide yes)
 			(show_name no)
@@
 		)
 		(property "Value" "SD_3V3"
-			(at 108.585 83.82 0)
+			(at 77.47 84.455 0)
 			(show_name no)
 			(do_not_autoplace no)
@@
 		)
 		(property "Footprint" ""
-			(at 108.585 88.9 0)
+			(at 77.47 89.535 0)
 			(hide yes)
 			(show_name no)
@@
 		)
 		(property "Datasheet" ""
-			(at 108.585 88.9 0)
+			(at 77.47 89.535 0)
 			(hide yes)
 			(show_name no)
@@
 		)
 		(property "Description" "Power symbol creates a global label with name \"+3V3\""
-			(at 108.585 88.9 0)
+			(at 77.47 89.535 0)
 			(hide yes)
 			(show_name no)
@@
 	(symbol
 		(lib_id "power:GND")
-		(at 108.585 116.84 0)
+		(at 77.47 117.475 0)
 		(unit 1)
 		(body_style 1)
@@
 		(fields_autoplaced yes)
 		(property "Reference" "#PWR05"
-			(at 108.585 123.19 0)
+			(at 77.47 123.825 0)
 			(hide yes)
 			(show_name no)
@@
 		)
 		(property "Value" "GND"
-			(at 108.585 121.92 0)
+			(at 77.47 122.555 0)
 			(show_name no)
 			(do_not_autoplace no)
@@
 		)
 		(property "Footprint" ""
-			(at 108.585 116.84 0)
+			(at 77.47 117.475 0)
 			(hide yes)
 			(show_name no)
@@
 		)
 		(property "Datasheet" ""
-			(at 108.585 116.84 0)
+			(at 77.47 117.475 0)
 			(hide yes)
 			(show_name no)
@@
 		)
 		(property "Description" "Power symbol creates a global label with name \"GND\" , ground"
-			(at 108.585 116.84 0)
+			(at 77.47 117.475 0)
 			(hide yes)
 			(show_name no)
@@
 	(symbol
 		(lib_id "power:PWR_FLAG")
-		(at 108.585 92.075 270)
+		(at 77.47 92.71 270)
 		(unit 1)
 		(body_style 1)
@@
 		(fields_autoplaced yes)
 		(property "Reference" "#FLG01"
-			(at 110.49 92.075 0)
+			(at 79.375 92.71 0)
 			(hide yes)
 			(show_name no)
@@
 		)
 		(property "Value" "PWR_FLAG"
-			(at 111.76 92.0749 90)
+			(at 80.645 92.7099 90)
 			(show_name no)
 			(do_not_autoplace no)
@@
 		)
 		(property "Footprint" ""
-			(at 108.585 92.075 0)
+			(at 77.47 92.71 0)
 			(hide yes)
 			(show_name no)
@@
 		)
 		(property "Datasheet" ""
-			(at 108.585 92.075 0)
+			(at 77.47 92.71 0)
 			(hide yes)
 			(show_name no)
@@
 		)
 		(property "Description" "Special symbol for telling ERC where power comes from"
-			(at 108.585 92.075 0)
+			(at 77.47 92.71 0)
 			(hide yes)
 			(show_name no)
@@
 	(symbol
 		(lib_id "power:PWR_FLAG")
-		(at 108.585 114.935 270)
+		(at 77.47 115.57 270)
 		(unit 1)
 		(body_style 1)
@@
 		(fields_autoplaced yes)
 		(property "Reference" "#FLG02"
-			(at 110.49 114.935 0)
+			(at 79.375 115.57 0)
 			(hide yes)
 			(show_name no)
@@
 		)
 		(property "Value" "PWR_FLAG"
-			(at 111.76 114.9349 90)
+			(at 80.645 115.5699 90)
 			(show_name no)
 			(do_not_autoplace no)
@@
 		)
 		(property "Footprint" ""
-			(at 108.585 114.935 0)
+			(at 77.47 115.57 0)
 			(hide yes)
 			(show_name no)
@@
 		)
 		(property "Datasheet" ""
-			(at 108.585 114.935 0)
+			(at 77.47 115.57 0)
 			(hide yes)
 			(show_name no)
@@
 		)
 		(property "Description" "Special symbol for telling ERC where power comes from"
-			(at 108.585 114.935 0)
-			(hide yes)
-			(show_name no)
+			(at 77.47 115.57 0)
+			(hide yes)
+			(show_name no)
